Commit message: Rewrite files

File: urdf/spot_zero.urdf (robot description, URDF)
Before this commit: robot bosdyn_spot, 26 links, 25 joints
Links:
- link base_link: geometry collision mesh filename=package://robot_dog_gait/meshes/base_link.STL scale=0.001 0.001 0.001; visual mesh filename=package://robot_dog_gait/meshes/base_link.STL scale=0.001 0.001 0.001
- link camera: geometry collision mesh filename=package://robot_dog_gait/meshes/camera.STL scale=0.001 0.001 0.001; visual mesh filename=package://robot_dog_gait/meshes/camera.STL scale=0.001 0.001 0.001
- link fl_hip_roll: geometry collision mesh filename=package://robot_dog_gait/meshes/fl_hip_roll.STL scale=0.001 0.001 0.001; visual mesh filename=package://robot_dog_gait/meshes/fl_hip_roll.STL scale=0.001 0.001 0.001
- link fl_hip_roll_connector: geometry collision mesh filename=package://robot_dog_gait/meshes/fl_hip_roll_connector.STL scale=0.001 0.001 0.001; visual mesh filename=package://robot_dog_gait/meshes/fl_hip_roll_connector.STL scale=0.001 0.001 0.001
- link fl_hip_yaw: geometry collision mesh filename=package://robot_dog_gait/meshes/fl_hip_yaw.STL scale=0.001 0.001 0.001; visual mesh filename=package://robot_dog_gait/meshes/fl_hip_yaw.STL scale=0.001 0.001 0.001
- link fl_hip_yaw_connector: geometry collision mesh filename=package://robot_dog_gait/meshes/fl_hip_yaw_connector.STL scale=0.001 0.001 0.001; visual mesh filename=package://robot_dog_gait/meshes/fl_hip_yaw_connector.STL scale=0.001 0.001 0.001
- link fl_knee: geometry collision mesh filename=package://robot_dog_gait/meshes/fl_knee.STL scale=0.001 0.001 0.001; collision sphere radius=0.0415
- link fr_hip_roll: geometry collision mesh filename=package://robot_dog_gait/meshes/fr_hip_roll.STL scale=0.001 0.001 0.001; visual mesh filename=package://robot_dog_gait/meshes/fr_hip_roll.STL scale=0.001 0.001 0.001
- link fr_hip_roll_connector: geometry collision mesh filename=package://robot_dog_gait/meshes/fr_hip_roll_connector.STL scale=0.001 0.001 0.001; visual mesh filename=package://robot_dog_gait/meshes/fr_hip_roll_connector.STL scale=0.001 0.001 0.001
- link fr_hip_yaw: geometry collision mesh filename=package://robot_dog_gait/meshes/fr_hip_yaw.STL scale=0.001 0.001 0.001; visual mesh filename=package://robot_dog_gait/meshes/fr_hip_yaw.STL scale=0.001 0.001 0.001
- link fr_hip_yaw_connector: geometry collision mesh filename=package://robot_dog_gait/meshes/fr_hip_yaw_connector.STL scale=0.001 0.001 0.001; visual mesh filename=package://robot_dog_gait/meshes/fr_hip_yaw_connector.STL scale=0.001 0.001 0.001
- link fr_knee: geometry collision mesh filename=package://robot_dog_gait/meshes/fr_knee.STL scale=0.001 0.001 0.001; collision sphere radius=0.0415
- link imu_sensor: geometry collision mesh filename=package://robot_dog_gait/meshes/imu_sensor.STL scale=0.001 0.001 0.001; visual mesh filename=package://robot_dog_gait/meshes/imu_sensor.STL scale=0.001 0.001 0.001
- link lidar: geometry collision mesh filename=package://robot_dog_gait/meshes/lidar.STL scale=0.001 0.001 0.001; visual mesh filename=package://robot_dog_gait/meshes/lidar.STL scale=0.001 0.001 0.001
- link rl_hip_roll: geometry collision mesh filename=package://robot_dog_gait/meshes/rl_hip_roll.STL scale=0.001 0.001 0.001; visual mesh filename=package://robot_dog_gait/meshes/rl_hip_roll.STL scale=0.001 0.001 0.001
- link rl_hip_roll_connector: geometry collision mesh filename=package://robot_dog_gait/meshes/rl_hip_roll_connector.STL scale=0.001 0.001 0.001; visual mesh filename=package://robot_dog_gait/meshes/rl_hip_roll_connector.STL scale=0.001 0.001 0.001
- link rl_hip_yaw: geometry collision mesh filename=package://robot_dog_gait/meshes/rl_hip_yaw.STL scale=0.001 0.001 0.001; visual mesh filename=package://robot_dog_gait/meshes/rl_hip_yaw.STL scale=0.001 0.001 0.001
- link rl_hip_yaw_connector: geometry collision mesh filename=package://robot_dog_gait/meshes/rl_hip_yaw_connector.STL scale=0.001 0.001 0.001; visual mesh filename=package://robot_dog_gait/meshes/rl_hip_yaw_connector.STL scale=0.001 0.001 0.001
- link rl_knee: geometry collision mesh filename=package://robot_dog_gait/meshes/rl_knee.STL scale=0.001 0.001 0.001; collision sphere radius=0.0415
- link rr_hip_roll: geometry collision mesh filename=package://robot_dog_gait/meshes/rr_hip_roll.STL scale=0.001 0.001 0.001; visual mesh filename=package://robot_dog_gait/meshes/rr_hip_roll.STL scale=0.001 0.001 0.001
- link rr_hip_roll_connector: geometry collision mesh filename=package://robot_dog_gait/meshes/rr_hip_roll_connector.STL scale=0.001 0.001 0.001; visual mesh filename=package://robot_dog_gait/meshes/rr_hip_roll_connector.STL scale=0.001 0.001 0.001
- link rr_hip_yaw: geometry collision mesh filename=package://robot_dog_gait/meshes/rr_hip_yaw.STL scale=0.001 0.001 0.001; visual mesh filename=package://robot_dog_gait/meshes/rr_hip_yaw.STL scale=0.001 0.001 0.001
- link rr_hip_yaw_connector: geometry collision mesh filename=package://robot_dog_gait/meshes/rr_hip_yaw_connector.STL scale=0.001 0.001 0.001; visual mesh filename=package://robot_dog_gait/meshes/rr_hip_yaw_connector.STL scale=0.001 0.001 0.001
- link rr_knee: geometry collision mesh filename=package://robot_dog_gait/meshes/rr_knee.STL scale=0.001 0.001 0.001; collision sphere radius=0.0415
